File: boards/keyboard/keyboard.kicad_sch (KiCad schematic)
At the start: 68 parts, among them J1 Keyboard Connector, T1 MountingHole_3.2mm_M3, T2 MountingHole_3.2mm_M3, T3 MountingHole_3.2mm_M3

Commit message: simplify/correct keyboard schematics
Parts:
- removed E5: A10, Connector_PinHeader_2.54mm:PinHeader_1x01_P2.54mm_Vertical, symbol Connector:Conn_01x01_Male
- removed E6: GND, Connector_PinHeader_2.54mm:PinHeader_1x01_P2.54mm_Vertical, symbol Connector:Conn_01x01_Male
- removed R24: 7K5, Resistor_THT:R_Axial_DIN0309_L9.0mm_D3.2mm_P12.70mm_Horizontal, symbol Device:R_Small_US
- removed RNalt1: 3K3, Resistor_THT:R_Array_SIP9, symbol Device:R_Network08
- removed Z7: 2758, Package_DIP:DIP-24_W15.24mm, symbol TopreLib:2758
- removed Z8: 4592, Package_DIP:DIP-40_W15.24mm_Socket, symbol ambassador:4592
- added Z7: 2758, Package_DIP:DIP-24_W15.24mm, symbol MyEprom:2758
- added Z8: AY-3-4592, Package_DIP:DIP-40_W15.24mm_Socket, symbol ambassador:4592_simple
- C14, C2, C6: symbol Keyboard-rescue:CP1_Small-Device -> Device:C_Polarized_Small_US
- C17: value 1uF tantalum -> 1uF; symbol Keyboard-rescue:CP1_Small-Device -> Device:C_Polarized_Small_US
- D1, D2, D3: symbol Keyboard-rescue:D_Small_ALT-Device -> Device:D_Small_Filled
- J1: symbol TopreLib:EdgeConn_02x18_Top_Bottom -> MyCardEdge:EdgeConn_02x18_Top_Bottom
- Z11, Z3: symbol Keyboard-rescue:74LS123-74xx -> 74xx:74LS123
Connections:
- net AKD: now also Z8.39 (AKD)
- net GND: now also Z7.12 (GND), Z7.18 (~{CE}), Z7.19 (AR), Z7.20 (~{OE}), Z8.1 (GND), Z8.13 (LO/RO)
- net KBINH: now also Z8.12 (KBINH)
- net Key Matrix/X0: now also Z8.17 (X0)
- net Key Matrix/X10: now also Z8.24 (X10)
- net Key Matrix/X11: now also Z8.25 (X11)
- net Key Matrix/X12: now also Z8.26 (X12)
- net Key Matrix/X13: now also Z8.27 (X13)
- net Key Matrix/X3: now also Z8.20 (X3)
- net Key Matrix/X4: now also Z8.21 (X4)
- net Key Matrix/X5: now also Z8.30 (X5)
- net Key Matrix/X6: now also Z8.32 (X6)
- net Key Matrix/X7: now also Z8.31 (X7)
- net Key Matrix/X8: now also Z8.22 (X8)
- net Key Matrix/X9: now also Z8.23 (X9)
- net VCC: now also Z7.21 (VPP), Z7.24 (VCC), Z8.40 (VCC)
- net X14: now also Z8.29 (X14)
- net ~{KPD}: now also Z8.35 (~{KPD})
- net ~{MATIN}: now also Z8.38 (~{MATIN})
- net at Z5.3: now also Z7.10 (D1)
- net at Z5.5: now also Z7.11 (D2)
- net at Z5.9: now also Z7.13 (D3)
- net at Z5.11: now also Z7.14 (D4)
- net at Z5.13: now also Z7.15 (D5)
- net at Z6.1: now also Z7.16 (D6)
- net at Z6.3: now also Z7.17 (D7)
- net at E3.1 (Pin_1), R7.2: now also Z7.22 (A9)
- net at Z5.1: now also Z7.9 (D0)
- net at Z10.11 (A): now also Z8.14 (YA)
- net at Z10.9 (C): now also Z8.15 (YC)
- net at Z10.10 (B): now also Z8.16 (YB)
- net at Z6.9: now also Z8.34 (SLI)
- net at C7.1, R9.2: now also Z8.36 (CLK)
- net at C6.1, D1.2 (A), R8.2: now also Z8.37 (~{POR})
- net +5P: now reaches R22.2, Z2.10 (~{S}), Z2.13 (~{R}), Z2.2 (D), Z2.4 (~{S}), Z3.10 (B), Z3.11 (Clr)
- new net: Z7.23 (A8), Z8.10 (D9)
- new net: Z7.8 (A0), Z8.2 (D1)
- new net: Z7.7 (A1), Z8.3 (D2)
- new net: Z7.6 (A2), Z8.4 (D3)
- new net: Z7.5 (A3), Z8.5 (D4)
- new net: Z7.4 (A4), Z8.6 (D5)
- new net: Z7.3 (A5), Z8.7 (D6)
- new net: Z7.2 (A6), Z8.8 (D7)
- new net: Z7.1 (A7), Z8.9 (D8)
Other:
- note added: "Caps Lock"
- note added: "Decode to ASCII (Inverted)"
- note added: "Inverters/Drivers"
- note added: "Power-On Reset"
- note added: "ROM region select"
- note added: "Sense amplification with custom I.C. See the circuit at the bottom of Fig. 1 of the AY-3-4592 datasheet for how it might be implemented."
- note added: "scan time 27ms"
- note removed: "10kOhm / 220pF gives 0.8MHz, scan time 27ms"
- note removed: "Jumper here to use lower half of ROM. Could add a key or switch to toggle between upper and lower halfs."
- note removed: "The 900C appears to be a custom linear (analog) IC. See the circuit at the bottom of Fig. 1 of the AY-3-4592 datasheet for how it might be implemented."
- moved on the sheet: C1, C10, C11, C12, C13, C14, C15, C16, C17, C2, C3, C4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

Commit message: keyboard schematic rev 1
Other:
- company: (none) -> Bradley Bell
- moved on the sheet: C10, C13, C14, C16, C17, C4, C7, C8, C9, CR4, D2, D3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
