File: boards/keyboard/key_matrix.kicad_sch (KiCad schematic)
At the start: 76 parts

Commit message: simplify/correct keyboard schematics
Parts:
- S39: footprint lib:NewKTPad_LED -> lib:KTCPad
Other:
- title: (none) -> Key Tronic Corp. 65-02163
Changed lines of the file:
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@@
 (kicad_sch (version 20211123) (generator eeschema)
   (paper "USLetter")
+  (title_block
+    (title "Key Tronic Corp. 65-02163")
+  )
   (junction (at 40.64 30.48) (diameter 0) (color 0 0 0 0)
   )
@@
   (symbol (lib_id "power:GND") (at 167.64 146.05 0) (unit 1)
     (in_bom yes) (on_board yes) (fields_autoplaced)
-    (property "Reference" "#PWR?" (id 0) (at 167.64 152.4 0)
+    (property "Reference" "#PWR0181" (id 0) (at 167.64 152.4 0)
       (effects (font (size 1.27 1.27)) hide)
     )
@@
       (effects (font (size 1.524 1.524)))
     )
-    (property "Footprint" "lib:NewKTPad_LED" (id 2) (at 160.02 67.31 0)
-      (effects (font (size 1.524 1.524)) hide)
-    )
+    (property "Footprint" "lib:KTCPad" (id 2) (at 160.02 67.31 0)
+      (effects (font (size 1.524 1.524)) hide)
+    )

Commit message: keyboard schematic rev 1
Other:
- company: (none) -> Bradley Bell
Changed lines of the file:
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@@
   (title_block
     (title "Key Tronic Corp. 65-02163")
+    (date "2023-04-23")
+    (rev "1")
+    (company "Bradley Bell")
   )
   (junction (at 40.64 30.48) (diameter 0) (color 0 0 0 0)
