File: boards/keyboard/keyboard.kicad_pcb (KiCad board)
At the start: 2 copper layers, 394.1 x 155.1 mm, 140 parts, among them J1 Keyboard Connector, T1 MountingHole_3.2mm_M3, T2 MountingHole_3.2mm_M3, T3 MountingHole_3.2mm_M3

Commit message: simplify/correct keyboard schematics
Parts:
- C17: value 1uF -> 1uF tantalum
- E3: value Conn_01x01_Male -> A9
- E4: value Conn_01x01_Male -> GND
- Z1: value 555 -> NE555P
- Z8: value AY-3-4592 -> 4592
Connections:
- net AKD renamed /AKD
- net KBD0 renamed /KBD0
- net KBD1 renamed /KBD1
- net KBD2 renamed /KBD2
- net KBD3 renamed /KBD3
- net KBD4 renamed /KBD4
- net KBD5 renamed /KBD5
- net KBD6 renamed /KBD6
- net KBD7 renamed /KBD7
- net KBINH renamed /KBINH
- net KBINT renamed /KBINT
- net MATSIG renamed /MATSIG
- net Net-(R22-Pad2) renamed +5P
- net UNUSED1 renamed /UNUSED1
- net UNUSED2 renamed /UNUSED2
- net X14 renamed /X14
- net ~{KPD} renamed /~{KPD}
- net ~{MATIN} renamed /~{MATIN}
Other:
- board text added: "github.com/btb/Telcon-Ambassador"
- board text removed: "btb"

Commit message: keyboard schematic rev 1
Parts:
- C17: value 1uF tantalum -> 1uF
- Z8: value 4592 -> AY-3-4592
Changed lines of the file:
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@@
       (effects (font (size 2.54 2.54) (thickness 0.254)) (justify mirror))
     )
-    (fp_text value "4592" (at 7.62 24.13 180) (layer "F.SilkS")
+    (fp_text value "AY-3-4592" (at 7.62 24.13 180) (layer "F.SilkS")
       (effects (font (size 1 1) (thickness 0.15)))
     )
@@
       (effects (font (size 1 1) (thickness 0.15)))
     )
-    (fp_text value "1uF tantalum" (at 6.35 0 90) (layer "F.SilkS")
-      (effects (font (size 1 1) (thickness 0.15)))
-    )
+    (fp_text value "1uF" (at 6.35 0 90) (layer "F.SilkS")
+      (effects (font (size 1 1) (thickness 0.15)))
+    )
