File: boards/mainboard/clock.kicad_sch (KiCad schematic)
At the start: 12 parts, among them U35 74163, U36 74163, U37 74163, U38 7420, U39 7408, U40 74S138, U41 7474, U43 7404, U62 7486

Commit message: organize mainboard schematic
Parts:
- removed C31, C32, C33: 220nF, ambassador:C_Disc_D4.3mm_W1.9mm_P6.35mm, symbol Device:C_Small
- removed unit 3 of U38
- removed unit 1 of U39
- removed unit 5 of U39
- removed unit 2 of U39
- removed unit 3 of U39
- removed U43: 7404, Package_DIP:DIP-14_W7.62mm, symbol 74xx:74LS04
Connections:
- net ~{OSCA}: now reaches U35.2 (CLK), U36.2 (CLK), U37.2 (CLK)
- net OSC/16 renamed OSC/16
- net OSC/4 renamed OSC/4
- net OSC/8 renamed OSC/8
- no-connect marks 32 -> 23
Other:
- moved on the sheet: U35, U36, U37, U38A, U38B, U39D, U40, U41A, U41B, U62B
