File: boards/mainboard/control.kicad_sch (KiCad schematic)
At the start: 11 parts, among them U10 7408, U11 7400, U13 74S139, U14 74S139, U43 7404, U51 7404, U64 7474, U65 7474, U66 7474, U67 7400

Commit message: organize mainboard schematic
Parts:
- removed C28: 220nF, ambassador:C_Disc_D4.3mm_W1.9mm_P6.35mm, symbol Device:C_Small
- removed unit 3 of U10
- removed unit 5 of U10
- removed unit 2 of U10
- removed unit 4 of U10
- removed unit 4 of U11
- removed unit 5 of U11
- removed unit 3 of U13
- removed U64, U65, U66: 7474, Package_DIP:DIP-14_W7.62mm, symbol 74xx:74LS74
- removed unit 5 of U67
- added U53: 7408, Package_DIP:DIP-14_W7.62mm, symbol 74xx:74LS08
- added U64, U65, U66: 7474, Package_DIP:DIP-14_W7.62mm, symbol 74xx:74LS74
- added unit 4 of U67
Connections:
- net GND: now also U66.2 (D)
- net U67P11: now also U67.11
- net VCC: now also U64.13 (~{R}), U65.10 (~{S}), U65.2 (D)
- new net: U53.6, U65.12 (D)
- new net: U65.3 (C), U65.9 (Q)
- new net: U64.2 (D), U65.6 (~{Q})
- new net: U64.3 (C), U64.9 (Q), U66.3 (C)
- new net: U65.5 (Q), U66.4 (~{S}), U67.13
- new net LC3: U53.5
- new net OSC/8: U64.11 (C), U65.11 (C)
- new net U64: U64.5 (Q)
- new net U66P6: U66.6 (~{Q})
- new net ~{DALOAD}: U53.4
- new net ~{DBE}: U64.12 (D)
- new net ~{DISP_EN}: U64.4 (~{S})
- new net ~{POS79}: U65.1 (~{R})
- new net ~{U64}: U64.6 (~{Q}), U67.12
- no-connect marks 17 -> 13
Other:
- note added: "$8-9000"
- note added: "$A-B000"
- note added: "$C-D000"
- note added: "$E-F000"
- note added: "$x000"
- note added: "$x004"
- note added: "$x008"
- note added: "$x00A"
- note removed: "$8000-$9000"
- note removed: "$A000,$B000"
- note removed: "$A000-$B000"
- note removed: "$A004,$B004"
- note removed: "$A008,$B008"
- note removed: "$A00A,$B00A"
- note removed: "$C000-$D000"
- note removed: "$E000-$F000"
- moved on the sheet: U10A, U11A, U11B, U13A, U13B, U14A, U43A, U51C, U67A, U67C
