File: boards/mainboard/d.kicad_sch (KiCad schematic)
At the start: 5 parts, among them U12 7404, U7 MC6800, U8 74LS241, U9 74LS241

Commit message: organize mainboard schematic
Parts:
- removed unit 4 of U12
- removed unit 5 of U12
- removed unit 3 of U12
- removed unit 7 of U12
- added unit 2 of U12
Connections:
- net ~{R}/W: now also U12.3
- new net R/~{W}: U12.4
- no-connect marks 13 -> 7
Other:
- moved on the sheet: RN1, U12A, U7, U8, U9
