File: boards/mainboard/ioc.kicad_sch (KiCad schematic)
At the start: 15 parts, among them P1 Presets, U12 7404, U70 6821, U71 6821, U76 7404

Commit message: organize mainboard schematic
Parts:
- removed C19, C5, C6: 220nF, ambassador:C_Disc_D4.3mm_W1.9mm_P6.35mm, symbol Device:C_Small
- removed U12: 7404, Package_DIP:DIP-14_W7.62mm, symbol 74xx:74LS04
- removed unit 6 of U76
- removed unit 7 of U76
Connections:
- net R/~{W}: now reaches U70.21 (R/~{W}), U71.21 (R/~{W})
- no-connect marks 10 -> 8
Other:
- moved on the sheet: LS1, P1, R2, R6, R7, R8, RN2, U71, U76A, U76B, U76C, U76D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
