File: boards/mainboard/mainboard.kicad_sch (KiCad schematic)
At the start: 8 parts, among them U43 7404, U44 12.5MHZ

Commit message: organize mainboard schematic
Parts:
- removed C15, C16, C17: 220nF, ambassador:C_Disc_D4.3mm_W1.9mm_P6.35mm, symbol Device:C_Small
- removed U43: 7404, Package_DIP:DIP-14_W7.62mm, symbol 74xx:74LS04
- removed U44: 12.5MHZ, Oscillator:Oscillator_DIP-14, symbol Oscillator:CXO_DIP14
- added RN4: R_Network09_Split, Resistor_THT:R_Array_SIP10, symbol Device:R_Network09_Split
Connections:
- net Horiz/HSYNC renamed HSYNC
- net IO/IND4 renamed IND4
- net IO/IND5 renamed IND5
- net IO/IND6 renamed IND6
- net Reset - Phi/RESET_SW renamed RESET_SW
- net Serial/CTSIND renamed CTSIND
- net Serial/RS232_CTS renamed RS232_CTS
- net Serial/RS232_DSR renamed RS232_DSR
- net Serial/RS232_DTR renamed RS232_DTR
- net Serial/RS232_RCK renamed RS232_RCK
- net Serial/RS232_RTS renamed RS232_RTS
- net Serial/RS232_RXD renamed RS232_RXD
- net Serial/RS232_TCK renamed RS232_TCK
- net Serial/RS232_TXD renamed RS232_TXD
- net Serial/RXIND renamed RXIND
- net Serial/TXIND renamed TXIND
- net Vert/~{VSYNC} renamed ~{VSYNC}
- net Video/VIDEO renamed VIDEO
- new net PULLUP: RN4.8 (R7.2)
- no-connect marks 1 -> 0
Other:
- sheet Display address counter renamed Display Address Counter
- sheet RAM renamed Memory
- sheet ROM renamed Firmware
- removed sheet Video
- added sheet Character Buffers (memcbuf.kicad_sch)
- added sheet Column Counters (column.kicad_sch)
- added sheet Line and Row Counter (line.kicad_sch)
- added sheet Memory Multiplexers (ram_multiplexers.kicad_sch)
- added sheet Other (unused.kicad_sch)
- added sheet Video Signal (video.kicad_sch)
- sheet CPU ports: added none; removed A0, A1, A10, A11, A12, A13, A14, A15, A2, A3, A4, A5, A6, A7, A8, A9, D0, D1, D2, D3, D4, D5, D6, D7, DBE, PHI1, PHI2, VMA, ~{IRQ}, ~{RESET}, ~{R}/W
- sheet Control ports: added none; removed A11, A12, A13, A14, A15, A2, A3, BAUD_SET, DBE, OSC/8, SERIAL_~{CS}, U67P11, VMA, ~{DBE}, ~{DISP_EN}, ~{IO_C_SEL}, ~{IO_D_SEL}, ~{RAM_EN}, ~{RAM_WE}, ~{ROM_EN}, ~{R}/W
- sheet Display Address Counter ports: added none; removed DA0, DA1, DA10, DA2, DA3, DA4, DA5, DA6, DA7, DA8, DA9, OSC, ~{DALOAD}, ~{DISP_EN}
- sheet Firmware ports: added none; removed A0, A1, A10, A11, A12, A2, A3, A4, A5, A6, A7, A8, A9, D0, D1, D2, D3, D4, D5, D6, D7, ~{RAM_WE}, ~{ROM_EN}, ~{R}/W
- sheet Horiz ports: added none; removed DBE, HBLANK, HSYNC, OSC, OSC/16, OSC/4, OSC/8, ROW_INC, U66P6, VRAM_EN, ~{DISP_EN}, ~{HBLANK}
- sheet IO ports: added none; removed A0, A1, D0, D1, D2, D3, D4, D5, D6, D7, DBE, IND4, IND5, IND6, RXRDY, TXRDY, ~{IO_C_SEL}, ~{IO_D_SEL}, ~{IRQ}, ~{RESET}, ~{R}/W
- sheet Memory ports: added none; removed A0, A1, A10, A11, A2, A3, A4, A5, A6, A7, A8, A9, D0, D1, D2, D3, D4, D5, D6, D7, DA0, DA1, DA10, DA2, DA3, DA4, DA5, DA6, DA7, DA8, DA9, DBE, ~{RAM_EN}, ~{RAM_WE}
- sheet Reset - Phi ports: added none; removed DBE, OSC/16, OSC/4, PHI1, PHI2, RESET, RESET_SW, ~{DBE}, ~{RESET}
- sheet Serial ports: added none; removed A0, A1, A2, A3, BAUD_SET, CTSIND, D0, D1, D2, D3, D4, D5, D6, D7, OSC/8, RESET, RS232_CTS, RS232_DSR, RS232_DTR, RS232_RCK, RS232_RTS, RS232_RXD, RS232_TCK, RS232_TXD, RXIND, RXRDY, SERIAL_~{CS}, TXIND, TXRDY, ~{R}/W
- sheet Vert ports: added none; removed ROW_INC, ~{DALOAD}, ~{VSYNC}
- moved on the sheet: A1, B1, JC1
