File: boards/mainboard/power.kicad_sch (KiCad schematic)
At the start: 26 parts, among them U11 7400, U68 74175, U69 5307, U73 75150_2, U74 8251, U75 7404, U77 75154, U78 75154, U79 75150_2, Y1 921.6KHZ

Commit message: organize mainboard schematic
Parts:
- removed C18, C20, C22: 220nF, ambassador:C_Disc_D4.3mm_W1.9mm_P6.35mm, symbol Device:C_Small
- removed unit 7 of U75
Connections:
- net OSC/8 renamed OSC/8
Other:
- moved on the sheet: C23, C24, C25, D2, JW2, R16, R17, R18, R3, R4, R5, R9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
