File: boards/mainboard/ram.kicad_sch (KiCad schematic)
At the start: 14 parts, among them U18 74157, U19 74157, U20 74157, U21 74S139, U22 MM2114, U23 MM2114, U24 MM2114, U26 MM2114, U27 MM2114, U28 MM2114

Commit message: organize mainboard schematic
Parts:
- removed C34, C35, C36, C40: 220nF, ambassador:C_Disc_D4.3mm_W1.9mm_P6.35mm, symbol Device:C_Small
- removed U18, U19, U20: 74157, Package_DIP:DIP-16_W7.62mm, symbol 74xx:74LS157
- removed unit 2 of U21
- removed unit 3 of U21
Connections:
- net RAMA6: now reaches U22.1 (A6), U23.1 (A6), U24.1 (A6), U26.1 (A6), U27.1 (A6), U28.1 (A6)
- net RAMA9: now reaches U22.15 (A9), U23.15 (A9), U24.15 (A9), U26.15 (A9), U27.15 (A9), U28.15 (A9)
- net RAMA8: now reaches U22.16 (A8), U23.16 (A8), U24.16 (A8), U26.16 (A8), U27.16 (A8), U28.16 (A8)
- net RAMA7: now reaches U22.17 (A7), U23.17 (A7), U24.17 (A7), U26.17 (A7), U27.17 (A7), U28.17 (A7)
- net RAMA5: now reaches U22.2 (A5), U23.2 (A5), U24.2 (A5), U26.2 (A5), U27.2 (A5), U28.2 (A5)
- net RAMA4: now reaches U22.3 (A4), U23.3 (A4), U24.3 (A4), U26.3 (A4), U27.3 (A4), U28.3 (A4)
- net RAMA3: now reaches U22.4 (A3), U23.4 (A3), U24.4 (A3), U26.4 (A3), U27.4 (A3), U28.4 (A3)
- net RAMA0: now reaches U22.5 (A0), U23.5 (A0), U24.5 (A0), U26.5 (A0), U27.5 (A0), U28.5 (A0)
- net RAMA1: now reaches U22.6 (A1), U23.6 (A1), U24.6 (A1), U26.6 (A1), U27.6 (A1), U28.6 (A1)
- net RAMA2: now reaches U22.7 (A2), U23.7 (A2), U24.7 (A2), U26.7 (A2), U27.7 (A2), U28.7 (A2)
- net RAMA11: now reaches U21.3 (A1)
- net RAMA10: now reaches U21.2 (A0)
- no-connect marks 8 -> 1
Other:
- moved on the sheet: U21A, U22, U23, U24, U26, U27, U28
