File: boards/mainboard/reset.kicad_sch (KiCad schematic)
At the start: 17 parts, among them Q1 2N3904, Q2 2N3904, Q3 2N3904, U72 7474, U80 7414

Commit message: organize mainboard schematic
Parts:
- removed C21, C27: 220nF, ambassador:C_Disc_D4.3mm_W1.9mm_P6.35mm, symbol Device:C_Small
- removed unit 2 of U72
- removed unit 3 of U72
- removed unit 3 of U80
- removed unit 6 of U80
- removed unit 7 of U80
- added U43: 7404, Package_DIP:DIP-14_W7.62mm, symbol 74xx:74LS04
- added U44: 12.5MHZ, Oscillator:Oscillator_DIP-14, symbol Oscillator:CXO_DIP14
Connections:
- net GND: now also U44.7 (GND)
- net VCC: now also U44.14 (Vcc)
- net OSC/16 renamed OSC/16
- net OSC/4 renamed OSC/4
- new net: U43.13, U44.8 (OUT)
- new net OSC: U43.11, U43.12, U43.9
- new net OSCB: U43.6
- new net ~{OSCA}: U43.10
- new net ~{OSCB}: U43.5, U43.8
- no-connect marks 12 -> 3
Other:
- moved on the sheet: C26, D17, Q1, Q2, Q3, R10, R11, R12, R13, R14, R15, R171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
