File: boards/mainboard/rom.kicad_sch (KiCad schematic)
At the start: 10 parts, among them U14 74S139, U3 6116, U4 6116, U5 2716, U6 2716

Commit message: organize mainboard schematic
Parts:
- removed C1, C2, C3, C4, C7: 220nF, ambassador:C_Disc_D4.3mm_W1.9mm_P6.35mm, symbol Device:C_Small
- removed unit 3 of U14
Other:
- moved on the sheet: U14B, U3, U4, U5, U6
