File: boards/mainboard/unused.kicad_sch (KiCad schematic)
At the start: 67 parts, among them U10 7408, U11 7400, U12 7404, U13 74S139, U14 74S139, U21 74S139, U33 7400, U34 7474, U38 7420, U39 7408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

Commit message: Update to KiCad 8
Parts:
- renumbered C17 to C18, C19 to C20, C21 to C22, U76 to U75
